Commit message: IR sensors added

File: src/turtlebot3/turtlebot3_description/urdf/turtlebot3_burger.gazebo.xacro (robot description, xacro)
@@ -136,3 +136,299 @@
       </plugin>
   </gazebo>
+  <gazebo reference="ir_1">
+   <sensor type="ray" name="TeraRanger">
+      <pose>0 0 0 0 0 0</pose>
+      <visualize>true</visualize>
+      <update_rate>50</update_rate>
+      <ray>
+         <scan>
+            <horizontal>
+               <samples>10</samples>
+               <resolution>1</resolution>
+               <min_angle>-0.14835</min_angle>
+               <max_angle>0.14835</max_angle>
+            </horizontal>
+            <vertical>
+               <samples>10</samples>
+               <resolution>1</resolution>
+               <min_angle>-0.14835</min_angle>
+               <max_angle>0.14835</max_angle>
+            </vertical>
+         </scan>
+         <range>
+            <min>0.01</min>
+            <max>2</max>
+            <resolution>0.02</resolution>
+         </range>
+      </ray>
+      <plugin filename="libgazebo_ros_range.so" name="gazebo_ros_range">
+         <gaussianNoise>0.005</gaussianNoise>
+         <alwaysOn>true</alwaysOn>
+         <updateRate>50</updateRate>
+         <topicName>sensor/ir_1</topicName>
+         <frameName>ir_1</frameName>
+         <radiation>INFRARED</radiation>
+         <fov>0.2967</fov>
+      </plugin>
+   </sensor>
+   </gazebo>
+     <gazebo reference="ir_2">
+      <sensor type="ray" name="TeraRanger">
+         <pose>0 0 0 0 0 0</pose>
+         <visualize>true</visualize>
+         <update_rate>50</update_rate>
+         <ray>
+            <scan>
+               <horizontal>
+                  <samples>10</samples>
+                  <resolution>1</resolution>
+                  <min_angle>-0.14835</min_angle>
+                  <max_angle>0.14835</max_angle>
+               </horizontal>
+               <vertical>
+                  <samples>10</samples>
+                  <resolution>1</resolution>
+                  <min_angle>-0.14835</min_angle>
+                  <max_angle>0.14835</max_angle>
+               </vertical>
+            </scan>
+            <range>
+               <min>0.01</min>
+               <max>2</max>
+               <resolution>0.02</resolution>
+            </range>
+         </ray>
+         <plugin filename="libgazebo_ros_range.so" name="gazebo_ros_range">
+            <gaussianNoise>0.005</gaussianNoise>
+            <alwaysOn>true</alwaysOn>
+            <updateRate>50</updateRate>
+            <topicName>sensor/ir_2</topicName>
+            <frameName>ir_2</frameName>
+            <radiation>INFRARED</radiation>
+            <fov>0.2967</fov>
+         </plugin>
+      </sensor>
+      </gazebo>
+      <gazebo reference="ir_3">
+       <sensor type="ray" name="TeraRanger">
+          <pose>0 0 0 0 0 0</pose>
+          <visualize>true</visualize>
+          <update_rate>50</update_rate>
+          <ray>
+             <scan>
+                <horizontal>
+                   <samples>10</samples>
+                   <resolution>1</resolution>
+                   <min_angle>-0.14835</min_angle>
+                   <max_angle>0.14835</max_angle>
+                </horizontal>
+                <vertical>
+                   <samples>10</samples>
+                   <resolution>1</resolution>
+                   <min_angle>-0.14835</min_angle>
+                   <max_angle>0.14835</max_angle>
+                </vertical>
+             </scan>
+             <range>
+                <min>0.01</min>
+                <max>2</max>
+                <resolution>0.02</resolution>
+             </range>
+          </ray>
+          <plugin filename="libgazebo_ros_range.so" name="gazebo_ros_range">
+             <gaussianNoise>0.005</gaussianNoise>
+             <alwaysOn>true</alwaysOn>
+             <updateRate>50</updateRate>
+             <topicName>sensor/ir_3</topicName>
+             <frameName>ir_3</frameName>
+             <radiation>INFRARED</radiation>
+             <fov>0.2967</fov>
+          </plugin>
+       </sensor>
+       </gazebo>
+       <gazebo reference="ir_4">
+        <sensor type="ray" name="TeraRanger">
+           <pose>0 0 0 0 0 0</pose>
+           <visualize>true</visualize>
+           <update_rate>50</update_rate>
+           <ray>
+              <scan>
+                 <horizontal>
+                    <samples>10</samples>
+                    <resolution>1</resolution>
+                    <min_angle>-0.14835</min_angle>
+                    <max_angle>0.14835</max_angle>
+                 </horizontal>
+                 <vertical>
+                    <samples>10</samples>
+                    <resolution>1</resolution>
+                    <min_angle>-0.14835</min_angle>
+                    <max_angle>0.14835</max_angle>
+                 </vertical>
+              </scan>
+              <range>
+                 <min>0.01</min>
+                 <max>2</max>
+                 <resolution>0.02</resolution>
+              </range>
+           </ray>
+           <plugin filename="libgazebo_ros_range.so" name="gazebo_ros_range">
+              <gaussianNoise>0.005</gaussianNoise>
+              <alwaysOn>true</alwaysOn>
+              <updateRate>50</updateRate>
+              <topicName>sensor/ir_4</topicName>
+              <frameName>ir_4</frameName>
+              <radiation>INFRARED</radiation>
+              <fov>0.2967</fov>
+           </plugin>
+        </sensor>
+        </gazebo>
+       <gazebo reference="ir_5">
+           <sensor type="ray" name="TeraRanger">
+              <pose>0 0 0 0 0 0</pose>
+              <visualize>true</visualize>
+              <update_rate>50</update_rate>
+              <ray>
+                 <scan>
+                    <horizontal>
+                       <samples>10</samples>
+                       <resolution>1</resolution>
+                       <min_angle>-0.14835</min_angle>
+                       <max_angle>0.14835</max_angle>
+                    </horizontal>
+                    <vertical>
+                       <samples>10</samples>
+                       <resolution>1</resolution>
+                       <min_angle>-0.14835</min_angle>
+                       <max_angle>0.14835</max_angle>
+                    </vertical>
+                 </scan>
+                 <range>
+                    <min>0.01</min>
+                    <max>2</max>
+                    <resolution>0.02</resolution>
+                 </range>
+              </ray>
+              <plugin filename="libgazebo_ros_range.so" name="gazebo_ros_range">
+                 <gaussianNoise>0.005</gaussianNoise>
+                 <alwaysOn>true</alwaysOn>
+                 <updateRate>50</updateRate>
+                 <topicName>sensor/ir_5</topicName>
+                 <frameName>ir_5</frameName>
+                 <radiation>INFRARED</radiation>
+                 <fov>0.2967</fov>
+              </plugin>
+           </sensor>
+           </gazebo>
+           <gazebo reference="ir_6">
+            <sensor type="ray" name="TeraRanger">
+               <pose>0 0 0 0 0 0</pose>
+               <visualize>true</visualize>
+               <update_rate>50</update_rate>
+               <ray>
+                  <scan>
+                     <horizontal>
+                        <samples>10</samples>
+                        <resolution>1</resolution>
+                        <min_angle>-0.14835</min_angle>
+                        <max_angle>0.14835</max_angle>
+                     </horizontal>
+                     <vertical>
+                        <samples>10</samples>
+                        <resolution>1</resolution>
+                        <min_angle>-0.14835</min_angle>
+                        <max_angle>0.14835</max_angle>
+                     </vertical>
+                  </scan>
+                  <range>
+                     <min>0.01</min>
+                     <max>2</max>
+                     <resolution>0.02</resolution>
+                  </range>
+               </ray>
+               <plugin filename="libgazebo_ros_range.so" name="gazebo_ros_range">
+                  <gaussianNoise>0.005</gaussianNoise>
+                  <alwaysOn>true</alwaysOn>
+                  <updateRate>50</updateRate>
+                  <topicName>sensor/ir_6</topicName>
+                  <frameName>ir_6</frameName>
+                  <radiation>INFRARED</radiation>
+                  <fov>0.2967</fov>
+               </plugin>
+            </sensor>
+            </gazebo>
+         <gazebo reference="ir_7">
+             <sensor type="ray" name="TeraRanger">
+                <pose>0 0 0 0 0 0</pose>
+                <visualize>true</visualize>
+                <update_rate>50</update_rate>
+                <ray>
+                   <scan>
+                      <horizontal>
+                         <samples>10</samples>
+                         <resolution>1</resolution>
+                         <min_angle>-0.14835</min_angle>
+                         <max_angle>0.14835</max_angle>
+                      </horizontal>
+                      <vertical>
+                         <samples>10</samples>
+                         <resolution>1</resolution>
+                         <min_angle>-0.14835</min_angle>
+                         <max_angle>0.14835</max_angle>
+                      </vertical>
+                   </scan>
+                   <range>
+                      <min>0.01</min>
+                      <max>2</max>
+                      <resolution>0.02</resolution>
+                   </range>
+                </ray>
+                <plugin filename="libgazebo_ros_range.so" name="gazebo_ros_range">
+                   <gaussianNoise>0.005</gaussianNoise>
+                   <alwaysOn>true</alwaysOn>
+                   <updateRate>50</updateRate>
+                   <topicName>sensor/ir_7</topicName>
+                   <frameName>ir_7</frameName>
+                   <radiation>INFRARED</radiation>
+                   <fov>0.2967</fov>
+                </plugin>
+             </sensor>
+             </gazebo>
+             <gazebo reference="ir_8">
+              <sensor type="ray" name="TeraRanger">
+                 <pose>0 0 0 0 0 0</pose>
+                 <visualize>true</visualize>
+                 <update_rate>50</update_rate>
+                 <ray>
+                    <scan>
+                       <horizontal>
+                          <samples>10</samples>
+                          <resolution>1</resolution>
+                          <min_angle>-0.14835</min_angle>
+                          <max_angle>0.14835</max_angle>
+                       </horizontal>
+                       <vertical>
+                          <samples>10</samples>
+                          <resolution>1</resolution>
+                          <min_angle>-0.14835</min_angle>
+                          <max_angle>0.14835</max_angle>
+                       </vertical>
+                    </scan>
+                    <range>
+                       <min>0.01</min>
+                       <max>2</max>
+                       <resolution>0.02</resolution>
+                    </range>
+                 </ray>
+                 <plugin filename="libgazebo_ros_range.so" name="gazebo_ros_range">
+                    <gaussianNoise>0.005</gaussianNoise>
+                    <alwaysOn>true</alwaysOn>
+                    <updateRate>50</updateRate>
+                    <topicName>sensor/ir_8</topicName>
+                    <frameName>ir_8</frameName>
+                    <radiation>INFRARED</radiation>
+                    <fov>0.2967</fov>
+                 </plugin>
+              </sensor>
+              </gazebo>
 </robot>

File: src/turtlebot3/turtlebot3_description/urdf/turtlebot3_burger.urdf.xacro (robot description, xacro)
@@ -140,3 +140,203 @@
     </inertial>
   </link>
+  <joint name="ir_1_joint" type="fixed">
+    <axis xyz="0 1 0" />
+    <origin rpy="0 0 -0.2627" xyz="0.09093 -0.02625 0.096" />
+    <parent link="base_link"/>
+    <child link="ir_1"/>
+ </joint>
+ <link name="ir_1">
+    <collision>
+      <origin xyz="0 0 0" rpy="0 0 0"/>
+      <geometry>
+        <box size="0.01 0.01 0.01"/>
+      </geometry>
+    </collision>
+    <visual>
+      <origin xyz="0 0 0" rpy="0 0 0"/>
+      <geometry>
+        <box size="0.01 0.01 0.01"/>
+      </geometry>
+    </visual>
+    <inertial>
+      <mass value="1e-5" />
+      <origin xyz="0 0 0" rpy="0 0 0"/>
+      <inertia ixx="1e-6" ixy="0" ixz="0" iyy="1e-6" iyz="0"      izz="1e-6" />
+    </inertial>
+ </link>
+ <joint name="ir_2_joint" type="fixed">
+   <axis xyz="0 1 0" />
+   <origin rpy="0 0 0.2627" xyz=" 0.09093 0.02625 0.096" />
+   <parent link="base_link"/>
+   <child link="ir_2"/>
+</joint>
+ <link name="ir_2">
+   <collision>
+     <origin xyz="0 0 0" rpy="0 0 0"/>
+     <geometry>
+       <box size="0.01 0.01 0.01"/>
+     </geometry>
+   </collision>
+   <visual>
+     <origin xyz="0 0 0" rpy="0 0 0"/>
+     <geometry>
+       <box size="0.01 0.01 0.01"/>
+     </geometry>
+   </visual>
+   <inertial>
+     <mass value="1e-5" />
+     <origin xyz="0 0 0" rpy="0 0 0"/>
+     <inertia ixx="1e-6" ixy="0" ixz="0" iyy="1e-6" iyz="0"      izz="1e-6" />
+   </inertial>
+</link>
+<joint name="ir_3_joint" type="fixed">
+  <axis xyz="0 1 0" />
+  <origin rpy="0 0 0.5236" xyz="0.0525 0.09093  0.096" />
+  <parent link="base_link"/>
+  <child link="ir_3"/>
+</joint>
+<link name="ir_3">
+  <collision>
+    <origin xyz="0 0 0" rpy="0 0 0"/>
+    <geometry>
+      <box size="0.01 0.01 0.01"/>
+    </geometry>
+  </collision>
+  <visual>
+    <origin xyz="0 0 0" rpy="0 0 0"/>
+    <geometry>
+      <box size="0.01 0.01 0.01"/>
+    </geometry>
+  </visual>
+  <inertial>
+    <mass value="1e-5" />
+    <origin xyz="0 0 0" rpy="0 0 0"/>
+    <inertia ixx="1e-6" ixy="0" ixz="0" iyy="1e-6" iyz="0"      izz="1e-6" />
+  </inertial>
+</link>
+<joint name="ir_4_joint" type="fixed">
+  <axis xyz="0 1 0" />
+  <origin rpy="0 0 -0.5236" xyz="0.0525 -0.09093  0.096" />
+  <parent link="base_link"/>
+  <child link="ir_4"/>
+</joint>
+<link name="ir_4">
+  <collision>
+    <origin xyz="0 0 0" rpy="0 0 0"/>
+    <geometry>
+      <box size="0.01 0.01 0.01"/>
+    </geometry>
+  </collision>
+  <visual>
+    <origin xyz="0 0 0" rpy="0 0 0"/>
+    <geometry>
+      <box size="0.01 0.01 0.01"/>
+    </geometry>
+  </visual>
+  <inertial>
+    <mass value="1e-5" />
+    <origin xyz="0 0 0" rpy="0 0 0"/>
+    <inertia ixx="1e-6" ixy="0" ixz="0" iyy="1e-6" iyz="0"      izz="1e-6" />
+  </inertial>
+</link>
+<joint name="ir_5_joint" type="fixed">
+  <axis xyz="0 1 0" />
+  <origin rpy="0 0 1.5708" xyz="0.0 0.105 0.096" />
+  <parent link="base_link"/>
+  <child link="ir_5"/>
+</joint>
+<link name="ir_5">
+  <collision>
+    <origin xyz="0 0 0" rpy="0 0 0"/>
+    <geometry>
+      <box size="0.01 0.01 0.01"/>
+    </geometry>
+  </collision>
+  <visual>
+    <origin xyz="0 0 0" rpy="0 0 0"/>
+    <geometry>
+      <box size="0.01 0.01 0.01"/>
+    </geometry>
+  </visual>
+  <inertial>
+    <mass value="1e-5" />
+    <origin xyz="0 0 0" rpy="0 0 0"/>
+    <inertia ixx="1e-6" ixy="0" ixz="0" iyy="1e-6" iyz="0"      izz="1e-6" />
+  </inertial>
+</link>
+<joint name="ir_6_joint" type="fixed">
+  <axis xyz="0 1 0" />
+  <origin rpy="0 0 -1.5708" xyz="0.0 -0.105 0.096" />
+  <parent link="base_link"/>
+  <child link="ir_6"/>
+</joint>
+<link name="ir_6">
+  <collision>
+    <origin xyz="0 0 0" rpy="0 0 0"/>
+    <geometry>
+      <box size="0.01 0.01 0.01"/>
+    </geometry>
+  </collision>
+  <visual>
+    <origin xyz="0 0 0" rpy="0 0 0"/>
+    <geometry>
+      <box size="0.01 0.01 0.01"/>
+    </geometry>
+  </visual>
+  <inertial>
+    <mass value="1e-5" />
+    <origin xyz="0 0 0" rpy="0 0 0"/>
+    <inertia ixx="1e-6" ixy="0" ixz="0" iyy="1e-6" iyz="0"      izz="1e-6" />
+  </inertial>
+</link>
+<joint name="ir_7_joint" type="fixed">
+  <axis xyz="0 1 0" />
+  <origin rpy="0 0 -2.879" xyz="-0.15 -0.02625 0.096" />
+  <parent link="base_link"/>
+  <child link="ir_7"/>
+</joint>
+<link name="ir_7">
+  <collision>
+    <origin xyz="0 0 0" rpy="0 0 0"/>
+    <geometry>
+      <box size="0.01 0.01 0.01"/>
+    </geometry>
+  </collision>
+  <visual>
+    <origin xyz="0 0 0" rpy="0 0 0"/>
+    <geometry>
+      <box size="0.01 0.01 0.01"/>
+    </geometry>
+  </visual>
+  <inertial>
+    <mass value="1e-5" />
+    <origin xyz="0 0 0" rpy="0 0 0"/>
+    <inertia ixx="1e-6" ixy="0" ixz="0" iyy="1e-6" iyz="0"      izz="1e-6" />
+  </inertial>
+</link>
+<joint name="ir_8_joint" type="fixed">
+  <axis xyz="0 1 0" />
+  <origin rpy="0 0 2.879" xyz="-0.15 0.02625 0.096" />
+  <parent link="base_link"/>
+  <child link="ir_8"/>
+</joint>
+<link name="ir_8">
+  <collision>
+    <origin xyz="0 0 0" rpy="0 0 0"/>
+    <geometry>
+      <box size="0.01 0.01 0.01"/>
+    </geometry>
+  </collision>
+  <visual>
+    <origin xyz="0 0 0" rpy="0 0 0"/>
+    <geometry>
+      <box size="0.01 0.01 0.01"/>
+    </geometry>
+  </visual>
+  <inertial>
+    <mass value="1e-5" />
+    <origin xyz="0 0 0" rpy="0 0 0"/>
+    <inertia ixx="1e-6" ixy="0" ixz="0" iyy="1e-6" iyz="0"      izz="1e-6" />
+  </inertial>
+</link>
 </robot>
